Commit message: aggiunta del palm

File: urdf/robot.urdf (robot description, URDF)
Before this commit: robot simple_example, 3 links, 2 joints
Links:
- added link palm_link, mass 0.2; collision box size=0.02 0.005 0.005; visual box size=0.02 0.005 0.005
Joints:
- added joint palm_joint: type continuous, parent third_link, child palm_link, origin xyz=0.0 0.0 0.1 rpy=0.0 0.0 0.0, axis 1 0 0

Commit message: aggiuni i link e joint di palmo e dito sinistro, posizione da sistemare

File: urdf/robot.urdf (robot description, URDF)
Before this commit: robot simple_example, 4 links, 3 joints
Links:
- added link left_finger, mass 0.2; collision box size=0.02 0.005 0.005; visual box size=0.02 0.005 0.005
Joints:
- added joint left_finger_joint: type continuous, parent third_link, child left_finger, origin xyz=-0.012 0.0 0.025 rpy=0.0 0.0 0.0, axis 1 0 0
- joint palm_joint: origin xyz=0.0 0.0 0.1 rpy=0.0 0.0 0.0 -> xyz=0.0 0.0 0.025 rpy=0.0 0.0 0.0
